File: Econet_ID_Extender_External/Econet_ID_Extender_External.kicad_pcb (KiCad board)
At the start: 2 copper layers, 42.9 x 23.2 mm, 7 parts, among them J1 Conn_02x06_Odd_Even, SW1 SW_DIP_x08

Commit message: Swap to standard 2.54 pitch ribbon
Parts:
- J1: footprint AliExpress_Stuff:MicroMatch-12p-SMD -> Connector_PinHeader_2.54mm:PinHeader_2x06_P2.54mm_Vertical_SMD
- moved J1 0.83 mm to (148.3, 91.3), turned to -90 degrees
Routing:
- net /E_GND: track 30.8 -> 0.00 mm
- net /E_SID_3: track 36.8 -> 8.97 mm
- net /E_SID_2: track 29.8 -> 8.97 mm
- net /E_SID_5: track 27.5 -> 8.97 mm, vias 1 -> 0
- net /E_SID_4: track 23.8 -> 8.97 mm
- net /E_AUD2: track 21.8 -> 31.7 mm, vias 2 -> 0
- net /E_SID_7: track 4.34 -> 12.3 mm
- net /E_SID_1: track 15.2 -> 8.97 mm
- net /E_SID_6: track 11.4 -> 17.1 mm, vias 1 -> 0
- net /E_AUD1: track 20.3 -> 25.2 mm
- net /E_SID_0: track 13.7 -> 8.97 mm
- net /E_AUD3: track 29.2 -> 33.5 mm, vias 2 -> 0
- added copper zone on B.Cu, net /E_GND
- removed copper zone on B.Cu, net (none)
- removed copper zone on F.Cu, net (none)
Other:
- board text added: "https://github.com/marrold/ BBC_Econet_ID_Extender v0.2"
