File: Econet_ID_Extender_External/Econet_ID_Extender_External.kicad_pcb (KiCad board)
At the start: 2 copper layers, 42.9 x 23.2 mm, 7 parts, among them J1 Conn_02x06_Odd_Even, SW1 SW_DIP_x08

Commit message: Add repo to silkscreen
Other:
- board text added: "https://github.com/marrold/ BBC_Econet_ID_Extender v0.1"
Changed lines of the file:
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@@
   (gr_line (start 128.809996 107.245782) (end 167.715782 107.245782) (layer "Edge.Cuts") (width 0.1))
   (gr_line (start 128.809996 84.035782) (end 167.715782 84.035782) (layer "Edge.Cuts") (width 0.1))
-  (gr_text "JLCJLCJLCJLC" (at 143.63 101.27) (layer "B.SilkS")
-    (effects (font (size 2 2) (thickness 0.4)) (justify mirror))
+  (gr_text "https://github.com/marrold/\nBBC_Econet_ID_Extender\nv0.1" (at 144.44 101.36) (layer "B.SilkS")
+    (effects (font (size 1 1) (thickness 0.2)) (justify mirror))
   )
   (gr_text "Econet ID\nExtender" (at 154.344132 91.069689) (layer "F.SilkS")
     (effects (font (size 2.2 2.2) (thickness 0.4)))
   )
+  (gr_text "JLCJLCJLCJLC" (at 143.63 101.27) (layer "F.SilkS")
+    (effects (font (size 1.5 1.5) (thickness 0.3)))
+  )
   (segment (start 148.29 91.52) (end 148.75 91.06) (width 0.25) (layer "B.Cu") (net 1))
