File: Econet_ID_Extender_External/Econet_ID_Extender_External.kicad_pcb (KiCad board)
At the start: 2 copper layers, 42.9 x 23.2 mm, 7 parts, among them J1 Conn_02x06_Odd_Even, SW1 SW_DIP_x08

Commit message: Fix volume pot orientation
Parts:
- moved RV1 5.07 mm to (161.9, 101.3), turned to 90 degrees
Connections:
- RV1 pad 1: /E_AUD1 -> /E_AUD3
- RV1 pad 3: /E_AUD3 -> /E_AUD1
Routing:
- net /E_AUD2: track 31.7 -> 26.6 mm
Other:
- board text added: "https://github.com/marrold/ BBC_Econet_ID_Extender v0.3"
- board text removed: "https://github.com/marrold/ BBC_Econet_ID_Extender v0.2"
Changed lines of the file:
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@@
   )
   (footprint "Potentiometer_THT:Potentiometer_Bourns_3386P_Vertical" (layer "F.Cu")
-    (at 156.812496 101.280782 -90)
+    (at 161.88 101.250782 90)
     (descr "Potentiometer, vertical, Bourns 3386P, https://www.bourns.com/pdfs/3386.pdf")
     (tags "Potentiometer vertical Bourns 3386P")
@@
     (fp_line (start -4.78 -7.305) (end -4.78 2.225) (layer "F.Fab") (width 0.1))
     (fp_circle (center -0.891 -2.54) (end 0.684 -2.54) (layer "F.Fab") (width 0.1) (fill none))
-    (pad "1" thru_hole circle (at 0 0 270) (size 1.44 1.44) (drill 0.8) (layers F&B.Cu *.Mask)
-      (net 1 "/E_AUD1") (pinfunction "1") (pintype "passive"))
-    (pad "2" thru_hole circle (at 2.54 -2.54 270) (size 1.44 1.44) (drill 0.8) (layers F&B.Cu *.Mask)
+    (pad "1" thru_hole circle (at 0 0 90) (size 1.44 1.44) (drill 0.8) (layers F&B.Cu *.Mask)
+      (net 3 "/E_AUD3") (pinfunction "1") (pintype "passive"))
+    (pad "2" thru_hole circle (at 2.54 -2.54 90) (size 1.44 1.44) (drill 0.8) (layers F&B.Cu *.Mask)
       (net 2 "/E_AUD2") (pinfunction "2") (pintype "passive"))
-    (pad "3" thru_hole circle (at 0 -5.08 270) (size 1.44 1.44) (drill 0.8) (layers F&B.Cu *.Mask)
-      (net 3 "/E_AUD3") (pinfunction "3") (pintype "passive"))
+    (pad "3" thru_hole circle (at 0 -5.08 90) (size 1.44 1.44) (drill 0.8) (layers F&B.Cu *.Mask)
+      (net 1 "/E_AUD1") (pinfunction "3") (pintype "passive"))
     (model "${KICAD6_3DMODEL_DIR}/Potentiometer_THT.3dshapes/Potentiometer_Bourns_3386P_Vertical.wrl"
       (offset (xyz 0 0 0))
@@
   (gr_line (start 128.809996 107.245782) (end 167.715782 107.245782) (layer "Edge.Cuts") (width 0.1))
   (gr_line (start 128.809996 84.035782) (end 167.715782 84.035782) (layer "Edge.Cuts") (width 0.1))
-  (gr_text "https://github.com/marrold/\nBBC_Econet_ID_Extender\nv0.2" (at 144.05 101.265782) (layer "B.SilkS")
+  (gr_text "https://github.com/marrold/\nBBC_Econet_ID_Extender\nv0.3" (at 144.05 101.265782) (layer "B.SilkS")
     (effects (font (size 1 1) (thickness 0.2)) (justify mirror))
   )
@@
   )
   (segment (start 156.97 101.123278) (end 156.812496 101.280782) (width 0.25) (layer "B.Cu") (net 1))
+  (segment (start 156.97 101.080782) (end 156.8 101.250782) (width 0.25) (layer "B.Cu") (net 1))
   (segment (start 146.992889 88.773532) (end 146.992889 88.347111) (width 0.25) (layer "B.Cu") (net 1))
-  (segment (start 156.97 87.87) (end 156.97 101.123278) (width 0.25) (layer "B.Cu") (net 1))
   (segment (start 155.65 86.55) (end 156.97 87.87) (width 0.25) (layer "B.Cu") (net 1))
   (segment (start 146.992889 88.347111) (end 148.79 86.55) (width 0.25) (layer "B.Cu") (net 1))
   (segment (start 148.79 86.55) (end 155.65 86.55) (width 0.25) (layer "B.Cu") (net 1))
-  (segment (start 159.352496 89.616806) (end 159.352496 103.820782) (width 0.25) (layer "B.Cu") (net 2))
+  (segment (start 156.97 87.87) (end 156.97 101.080782) (width 0.25) (layer "B.Cu") (net 1))
   (segment (start 147.125922 86.100499) (end 155.836189 86.100499) (width 0.25) (layer "B.Cu") (net 2))
+  (segment (start 159.34 89.629302) (end 159.34 98.710782) (width 0.25) (layer "B.Cu") (net 2))
   (segment (start 144.452889 88.773532) (end 147.125922 86.100499) (width 0.25) (layer "B.Cu") (net 2))
+  (segment (start 159.352496 89.616806) (end 159.34 89.629302) (width 0.25) (layer "B.Cu") (net 2))
   (segment (start 155.836189 86.100499) (end 159.352496 89.616806) (width 0.25) (layer "B.Cu") (net 2))
   (segment (start 156.022378 85.650998) (end 161.892496 91.521116) (width 0.25) (layer "B.Cu") (net 3))
-  (segment (start 161.892496 91.521116) (end 161.892496 101.280782) (width 0.25) (layer "B.Cu") (net 3))
+  (segment (start 161.892496 91.521116) (end 161.88 91.533612) (width 0.25) (layer "B.Cu") (net 3))
+  (segment (start 161.88 91.533612) (end 161.88 101.250782) (width 0.25) (layer "B.Cu") (net 3))
   (segment (start 141.912889 88.773532) (end 145.035423 85.650998) (width 0.25) (layer "B.Cu") (net 3))
   (segment (start 145.035423 85.650998) (end 156.022378 85.650998) (width 0.25) (layer "B.Cu") (net 3))
